Commit message: split main file up into file includes

File: src/my_robot_description/urdf/mobile_base.xml.xacro (robot description, xacro)
@@ -1,15 +1,10 @@
 <?xml version="1.0"?>
-<!-- create the robot -->
-<robot name="my_robot">
-    <!-- defining colours for robot -->
-    <material name="blue">
-        <color rgba="0 0 0.5 1"/>
-    </material>
-    <material name="grey">
-        <color rgba="0.5 0.5 0.5 1"/>
-    </material>
-    <material name="red">
-        <color rgba="0.5 0 0 1"/>
-    </material>
+<robot xmlns:xacro="http://www.ros.org/wiki/xacro">
+    <!-- variables reused amount robot parts -->
+    <xacro:property name="base_length" value="0.6" />
+    <xacro:property name="base_width" value="0.4" />
+    <xacro:property name="base_height" value="0.2" />
+    <xacro:property name="wheel_radius" value="0.1" />
+    <xacro:property name="wheel_length" value="0.05" />
     <!-- base footprint to lift the entire model above the ground -->
     <link name="base_footprint">
@@ -21,39 +16,33 @@
             <geometry>
                 <!-- length, width, height in meters -->
-                <box size="0.6 0.4 0.2"/>
+                <box size="${base_length} ${base_width} ${base_height}"/>
             </geometry>
             <!-- roll, pitch, yaw ie rotation on the x, y and z axis respective -->
-            <origin xyz="0 0 0.1" rpy="0 0 0"/>
+            <origin xyz="0 0 ${base_height / 2.0}" rpy="0 0 0"/>
             <!-- use the mertial tag declared above -->
             <material name="blue" />
         </visual>
     </link>
-    <!-- right wheel link -->
-    <link name="right_wheel_link">
-        <visual>
-            <geometry>
-                <cylinder radius="0.1" length="0.05"/>
-            </geometry>
-            <origin xyz="0 0 0" rpy="1.57 0 0" />
-            <material name="grey" />
-        </visual>
-    </link>
     <!-- left wheel link -->
-    <link name="left_wheel_link">
-        <visual>
-            <geometry>
-                <cylinder radius="0.1" length="0.05"/>
-            </geometry>
-            <origin xyz="0 0 0" rpy="1.57 0 0" />
-            <material name="grey" />
-        </visual>
-    </link>
+    <xacro:macro name="wheel_link" params="prefix">
+        <link name="${prefix}_wheel_link">
+            <visual>
+                <geometry>
+                    <cylinder radius="${wheel_radius}" length="${wheel_length}"/>
+                </geometry>
+                <origin xyz="0 0 0" rpy="${pi / 2.0} 0 0" />
+                <material name="grey" />
+            </visual>
+        </link>
+    </xacro:macro>
+    <xacro:wheel_link prefix="right" />
+    <xacro:wheel_link prefix="left" />
     <!-- front wheel link -->
     <link name="caster_wheel_link">
         <visual>
             <geometry>
-                <sphere radius="0.05" />
+                <sphere radius="${wheel_radius / 2.0}" />
             </geometry>
-            <origin xyz="0 0 -0.025" rpy="0 0 0" />
+            <origin xyz="0 0 0" rpy="0 0 0" />
             <material name="grey" />
         </visual>
@@ -64,5 +53,5 @@
         <parent link="base_footprint"/>
         <child link="base_link" />
-        <origin xyz="0 0 0.1" rpy="0 0 0" />
+        <origin xyz="0 0 ${wheel_radius}" rpy="0 0 0" />
         <axis xyz="0 1 0" />
     </joint>
@@ -71,5 +60,5 @@
         <parent link="base_link"/>
         <child link="right_wheel_link" />
-        <origin xyz="-0.15 -0.225 0" rpy="0 0 0" />
+        <origin xyz="${-base_length / 4.0} ${-(base_width + wheel_length) / 2.0} 0" rpy="0 0 0" />
         <axis xyz="0 1 0" />
     </joint>
@@ -78,5 +67,5 @@
         <parent link="base_link"/>
         <child link="left_wheel_link" />
-        <origin xyz="-0.15 0.225 0" rpy="0 0 0" />
+        <origin xyz="${-base_length / 4.0} ${(base_width + wheel_length) / 2.0} 0" rpy="0 0 0" />
         <axis xyz="0 1 0" />
     </joint>
@@ -85,5 +74,5 @@
         <parent link="base_link"/>
         <child link="caster_wheel_link" />
-        <origin xyz="0.2 0 0" rpy="0 0 0" />
+        <origin xyz="${base_length / 3.0} 0 ${-wheel_radius / 2.0}" rpy="0 0 0" />
         <axis xyz="0 1 0" />
     </joint>
