Commit message: add camera sensor to gazebo plugin

File: src/my_robot_description/urdf/camera.xml.xacro (robot description, xacro)
@@ -22,5 +22,16 @@
         <parent link="base_link" />
         <child link="camera_link" />
-        <origin xyz="${base_length + camera_length / 2.0} 0 ${base_height / 2.0}" rpy="0 0 0" />
+        <origin xyz="${(base_length + camera_length) / 2.0} 0 ${base_height / 2.0}" rpy="0 0 0" />
     </joint>
+    <gazebo reference="camera_link">
+        <material>Gabezo/Grey</material>
+        <sensor name="camera_sensor" type="camera">
+            <pose>0 0 0 0 0 0</pose>
+            <visualize>true</visualize>
+            <update_rate>10.0</update_rate>
+            <plugin name="camera_controller" filename="libgazebo_ros_camera.so">
+                <frame_name>camera_link</frame_name>
+              </plugin>
+        </sensor>
+    </gazebo>
 </robot>

Commit message: fix issue to do with camera inconsistancy with ros and opencv

File: src/my_robot_description/urdf/camera.xml.xacro (robot description, xacro)
@@ -24,4 +24,14 @@
         <origin xyz="${(base_length + camera_length) / 2.0} 0 ${base_height / 2.0}" rpy="0 0 0" />
     </joint>
+    <joint name="camera_optical_joint" type="fixed">
+        <!-- these values have to be these values otherwise the gazebo camera
+            image won't be aligned properly with the frame it is supposedly
+            originating from -->
+        <origin xyz="0 0 0" rpy="${-pi/2} 0 ${-pi/2}"/>
+        <parent link="camera_link"/>
+        <child link="camera_link_optical"/>
+    </joint>
+    <link name="camera_link_optical">
+    </link>
     <gazebo reference="camera_link">
         <material>Gabezo/Grey</material>
