Commit message: achieve the correct rviz urdf

File: src/my_robot_description/urdf/arm.xml.xacro (robot description, xacro)
@@ -34,5 +34,5 @@
                 <cylinder radius="${cylinder_radius}" length="${cylinder_length}" />
             </geometry>
-            <origin xyz="0 0 0" rpy="0 0 0" />
+            <origin xyz="0 0 ${cylinder_length / 2}" rpy="0 0 0" />
             <material name="yellow" />
         </visual>
@@ -51,5 +51,5 @@
                 <cylinder radius="${cylinder_radius}" length="${cylinder_length}" />
             </geometry>
-            <origin xyz="0 0 0" rpy="0 0 0" />
+            <origin xyz="0 0 ${cylinder_length / 2}" rpy="0 0 0" />
             <material name="orange" />
         </visual>
@@ -73,5 +73,5 @@
         <parent link="arm_base_link" />
         <child link="forearm_link" />
-        <origin xyz="0 0 ${(cylinder_length / 2 + cuboid_height)}" rpy="0 0 0" />
+        <origin xyz="0 0 ${cuboid_height}" rpy="0 0 0" />
         <axis xyz="0 1 0" />
         <dynamics friction="0.05" damping="0.1" />

File: src/my_robot_description/urdf/arm_gazebo.xml.xacro (robot description, xacro)
@@ -15,7 +15,7 @@
             <update_rate>2</update_rate>
             <!-- name of joints in the model whose states will be published. -->
-            <base_joint>arm_base_joint</base_joint>
-            <forearm_joint>arm_base_forearm_joint</forearm_joint>
-            <hand_joint>forearm_hand_joint</hand_joint>
+            <joint_name>arm_base_joint</joint_name>
+            <joint_name>arm_base_forearm_joint</joint_name>
+            <joint_name>forearm_hand_joint</joint_name>
         </plugin>
         <plugin name="joint_pose_trajectory" filename="libgazebo_ros_joint_pose_trajectory.so">

Commit message: combine robot arm and turtlebot

File: src/my_robot_description/urdf/arm.xml.xacro (robot description, xacro)
@@ -11,5 +11,4 @@
     <xacro:property name="cylinder_radius" value="0.02" />
     <!-- robot links -->
-    <link name="arm_base_footprint_link" />
     <link name="arm_base_link">
         <visual>
@@ -26,5 +25,5 @@
             <origin xyz="0 0 ${cuboid_height / 2}" rpy="0 0 0" />
         </collision>
-        <xacro:cuboid_inertia m="${cuboid_mass}" l="${cuboid_length}" w="${cuboid_width}" h="${cuboid_height}"
+        <xacro:cuboid_inertia m="${cuboid_mass}" l="${cuboid_length * 2}" w="${cuboid_width * 2}" h="${cuboid_height * 2}"
                               xyz="0 0 ${cuboid_height / 2.0}" rpy="0 0 0" />
     </link>
@@ -34,5 +33,5 @@
                 <cylinder radius="${cylinder_radius}" length="${cylinder_length}" />
             </geometry>
-            <origin xyz="0 0 ${cylinder_length / 2}" rpy="0 0 0" />
+            <origin xyz="0 0 ${(cylinder_length / 2)}" rpy="0 0 0" />
             <material name="yellow" />
         </visual>
@@ -41,8 +40,8 @@
                 <cylinder radius="${cylinder_radius}" length="${cylinder_length}" />
             </geometry>
-            <origin xyz="0 0 0" rpy="0 0 0" />
+            <origin xyz="0 0 ${(cylinder_length / 2)}" rpy="0 0 0" />
         </collision>
-        <xacro:cylinder_inertia m="${cylinder_mass}" r="${cylinder_radius}" h="${cylinder_length}"
-                                xyz="0 0 ${cylinder_length / 2}" rpy="0 0 0" />
+        <xacro:cylinder_inertia m="${cylinder_mass}" r="${cylinder_radius * 2}" h="${cylinder_length * 2}"
+                                xyz="0 0 ${(cylinder_length / 2)}" rpy="0 0 0" />
     </link>
     <link name="hand_link">
@@ -51,5 +50,5 @@
                 <cylinder radius="${cylinder_radius}" length="${cylinder_length}" />
             </geometry>
-            <origin xyz="0 0 ${cylinder_length / 2}" rpy="0 0 0" />
+            <origin xyz="0 0 ${(cylinder_length / 2)}" rpy="0 0 0" />
             <material name="orange" />
         </visual>
@@ -58,15 +57,10 @@
                 <cylinder radius="${cylinder_radius}" length="${cylinder_length}" />
             </geometry>
-            <origin xyz="0 0 0" rpy="0 0 0" />
+            <origin xyz="0 0 ${(cylinder_length / 2)}" rpy="0 0 0" />
         </collision>
-        <xacro:cylinder_inertia m="${cylinder_mass}" r="${cylinder_radius}" h="${cylinder_length}"
-                                xyz="0 0 ${cylinder_length / 2}" rpy="0 0 0" />
+        <xacro:cylinder_inertia m="${cylinder_mass}" r="${cylinder_radius * 2}" h="${cylinder_length * 2}"
+                                xyz="0 0 ${(cylinder_length / 2)}" rpy="0 0 0" />
     </link>
     <!-- arm joints -->
-    <joint name="arm_base_joint" type="fixed">
-        <parent link="arm_base_footprint_link" />
-        <child link="arm_base_link" />
-        <origin xyz="0 0 ${cuboid_height}" rpy="0 0 0"/>
-    </joint>
     <joint name="arm_base_forearm_joint" type="revolute">
         <limit lower="0" upper="${pi / 2}" effort="100" velocity="100" />

File: src/my_robot_description/urdf/my_robot.urdf.xacro (robot description, xacro)
@@ -4,4 +4,11 @@
     <xacro:include filename="mobile_base.xacro" />
     <xacro:include filename="mobile_base_gazebo.xml.xacro"/>
+    <xacro:include filename="arm.xml.xacro" />
+    <xacro:include filename="arm_gazebo.xml.xacro" />
+    <joint name="mobile_base_arm_joint" type="fixed">
+        <parent link="base_link" />
+        <child link="arm_base_link" />
+        <origin xyz="${base_length / 4.0} 0 ${base_height}" rpy="0 0 0" />
+    </joint>
     <xacro:include filename="camera.xml.xacro"/>
 </robot>
